Commit message: steering controllers working

File: fake_car.urdf (robot description, URDF)
Before this commit: robot fake_car, 7 links, 6 joints
Joints:
- joint back_left_wheel_joint: limit (none) -> effort=10000 velocity=100
- joint front_left_wheel_steer_joint: limit (none) -> lower=-1 upper=1 effort=1 velocity=5; type continuous -> revolute
- joint front_right_wheel_steer_joint: limit (none) -> lower=-1 upper=1 effort=1 velocity=5; type continuous -> revolute

Commit message: back wheels working

File: fake_car.urdf (robot description, URDF)
Before this commit: robot fake_car, 7 links, 6 joints
Joints:
- joint back_left_wheel_joint: limit effort=10000 velocity=100 -> effort=10000 velocity=500
- joint back_right_wheel_joint: limit (none) -> effort=10000 velocity=500

Commit message: added laser

File: fake_car.urdf (robot description, URDF)
Before this commit: robot fake_car, 7 links, 6 joints
Links:
- added link laser_scanner_link, mass 1e-5; collision box size=.127 0.1016 0.0508; visual box size=.127 0.1016 0.0508
Joints:
- added joint laser_scanner_joint: type fixed, parent base_link, child laser_scanner_link, origin xyz=0.1397 0 0.2159 rpy=0 0 0

Commit message: updated with xacro

File: fake_car.urdf (robot description, URDF)
Before this commit: robot fake_car, 8 links, 7 joints
Links:
- added link back_left_wheel_shock, mass 0.01; collision cylinder length=0.2 radius=0.01; visual cylinder length=0.2 radius=0.01
- added link back_right_wheel_shock, mass 0.01; collision cylinder length=0.2 radius=0.01; visual cylinder length=0.2 radius=0.01
- added link chassis_link, mass 2.6; collision box size=0.3429 0.25 0.06; visual box size=0.3429 0.25 0.06
- added link front_left_wheel_shock, mass 0.01; collision cylinder length=0.2 radius=0.01; visual cylinder length=0.2 radius=0.01
- added link front_right_wheel_shock, mass 0.01; collision cylinder length=0.2 radius=0.01; visual cylinder length=0.2 radius=0.01
- link base_link: mass 1.0 -> 0.01; geometry collision cylinder length=0.2 radius=0.01; visual cylinder length=0.2 radius=0.01
- link front_left_wheel_steer: geometry collision cylinder length=0.01 radius=0.01; visual cylinder length=0.01 radius=0.01
- link front_right_wheel_steer: geometry collision cylinder length=0.01 radius=0.01; visual cylinder length=0.01 radius=0.01
Joints:
- added joint back_left_shock_joint: type prismatic, parent base_link, child back_left_wheel_shock, origin xyz=0 0.125  -0.045 rpy=0 0 0, axis 0 0 1, limit lower=0 upper=0.09 effort=100 velocity=100
- added joint back_right_shock_joint: type prismatic, parent base_link, child back_right_wheel_shock, origin xyz=0 -0.125 -0.045 rpy=0 0 0, axis 0 0 1, limit lower=0 upper=0.09 effort=100 velocity=100
- added joint chassis_joint: type fixed, parent base_link, child chassis_link, origin xyz=0.17145 0 0.02 rpy=0 0 0
- added joint front_left_shock_joint: type prismatic, parent base_link, child front_left_wheel_shock, origin xyz=0.3429 0.125  -0.045 rpy=0 0 0, axis 0 0 1, limit lower=0 upper=0.09 effort=100 velocity=100
- added joint front_right_shock_joint: type prismatic, parent base_link, child front_right_wheel_shock, origin xyz=0.3429 -0.125 -0.045 rpy=0 0 0, axis 0 0 1, limit lower=0 upper=0.09 effort=100 velocity=100
- joint back_left_wheel_joint: origin xyz=0 0.125 0 rpy=-1.5708 0 0 -> xyz=0 0 0 rpy=-1.57079632679 0 0; parent base_link -> back_left_wheel_shock
- joint back_right_wheel_joint: origin xyz=0 -0.125 0.0 rpy=-1.5708 0 0 -> xyz=0 0 0 rpy=-1.57079632679 0 0; parent base_link -> back_right_wheel_shock
- joint front_left_wheel_joint: origin xyz=0 0 0 rpy=-1.5708 0 0 -> xyz=0 0 0 rpy=-1.57079632679 0 0
- joint front_left_wheel_steer_joint: origin xyz=0.3429 0.125 0 rpy=0 0 0 -> xyz=0 0 0 rpy=0 0 0; parent base_link -> front_left_wheel_shock
- joint front_right_wheel_joint: origin xyz=0 0 0 rpy=-1.5708 0 0 -> xyz=0 0 0 rpy=-1.57079632679 0 0
- joint front_right_wheel_steer_joint: origin xyz=0.3429 -0.125 0 rpy=0 0 0 -> xyz=0 0 0 rpy=0 0 0; parent base_link -> front_right_wheel_shock
